File: board/solohm.sch (EAGLE design)
At the start: 108 parts, among them Q1 1984620, Q2 1984620, Q3 1984620, Q4 1984620, Q5 1984620, Q6 1984620, Q7 1984620, Q8 1984620, U1 20, U10 AP2210K-5.0TRG1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

Commit message: here's the v0.1 hardware version, sent this to board house for fab
Parts:
- added R34, R35: 10K, holla:R-US_R0603
Connections:
- net DISPLAYRESET: now also R35.2
- net GND: now also R35.1
- net THERMOCOUPLECS: now also R34.1
- net V3.3: now also R34.2
Other:
- moved on the sheet: C9, TC-K, U5
Changed lines of the file:
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@@
 <part name="C10" library="holla" deviceset="C" device="-USC0603" value=".1u"/>
 <part name="GND8" library="holla" deviceset="GND" device=""/>
-<part name="IPANEL" library="holla" deviceset="TESTPOINT" device="THRU"/>
+<part name="IPANEL" library="holla" deviceset="TESTPOINT" device="THRU" value=""/>
 <part name="PHOTOCELL" library="holla" deviceset="1984617" device="" value=""/>
 <part name="R13" library="holla" deviceset="R" device="-US_R0603" value="47K"/>
@@
 <part name="TC-K" library="holla" deviceset="M02" device="-1984617"/>
 <part name="JP3" library="holla" deviceset="M05" device="PTH"/>
+<part name="R34" library="holla" deviceset="R" device="-US_R0603" value="10K"/>
+<part name="R35" library="holla" deviceset="R" device="-US_R0603" value="10K"/>
 </parts>
 <sheets>
@@
 <instance part="FRAME3" gate="G$1" x="0" y="0"/>
 <instance part="FRAME3" gate="G$2" x="172.72" y="0"/>
-<instance part="U5" gate="G$1" x="210.82" y="180.34"/>
-<instance part="GND7" gate="1" x="195.58" y="162.56"/>
-<instance part="C9" gate="G$1" x="193.04" y="172.72"/>
+<instance part="U5" gate="G$1" x="193.04" y="180.34"/>
+<instance part="GND7" gate="1" x="177.8" y="162.56"/>
+<instance part="C9" gate="G$1" x="175.26" y="172.72"/>
 <instance part="R11" gate="G$1" x="22.86" y="200.66" rot="R90"/>
 <instance part="R12" gate="G$1" x="22.86" y="185.42" rot="R90"/>
@@
 <instance part="GND17" gate="1" x="241.3" y="114.3"/>
 <instance part="R24" gate="G$1" x="251.46" y="134.62" rot="R90"/>
-<instance part="GND15" gate="1" x="203.2" y="68.58"/>
+<instance part="GND15" gate="1" x="203.2" y="60.96"/>
 <instance part="GND14" gate="1" x="243.84" y="48.26" rot="MR0"/>
 <instance part="D10" gate="G$1" x="246.38" y="175.26"/>
@@
 <instance part="C26" gate="G$1" x="177.8" y="114.3"/>
 <instance part="U12" gate="G$1" x="119.38" y="30.48" rot="MR0"/>
-<instance part="TC-K" gate="G$1" x="180.34" y="180.34"/>
+<instance part="TC-K" gate="G$1" x="162.56" y="180.34"/>
 <instance part="JP3" gate="G$1" x="190.5" y="76.2"/>
+<instance part="R34" gate="G$1" x="218.44" y="185.42" rot="R90"/>
+<instance part="R35" gate="G$1" x="228.6" y="73.66" rot="R90"/>
 </instances>
 <busses>
@@
 <pinref part="U5" gate="G$1" pin="GND"/>
 <pinref part="GND7" gate="1" pin="GND"/>
-<wire x1="198.12" y1="175.26" x2="195.58" y2="175.26" width="0.1524" layer="91"/>
-<wire x1="195.58" y1="175.26" x2="195.58" y2="167.64" width="0.1524" layer="91"/>
+<wire x1="180.34" y1="175.26" x2="177.8" y2="175.26" width="0.1524" layer="91"/>
+<wire x1="177.8" y1="175.26" x2="177.8" y2="167.64" width="0.1524" layer="91"/>
 <pinref part="C9" gate="G$1" pin="2"/>
-<wire x1="195.58" y1="167.64" x2="195.58" y2="165.1" width="0.1524" layer="91"/>
-<wire x1="193.04" y1="170.18" x2="193.04" y2="167.64" width="0.1524" layer="91"/>
-<wire x1="193.04" y1="167.64" x2="195.58" y2="167.64" width="0.1524" layer="91"/>
-<junction x="195.58" y="167.64"/>
+<wire x1="177.8" y1="167.64" x2="177.8" y2="165.1" width="0.1524" layer="91"/>
+<wire x1="175.26" y1="170.18" x2="175.26" y2="167.64" width="0.1524" layer="91"/>
+<wire x1="175.26" y1="167.64" x2="177.8" y2="167.64" width="0.1524" layer="91"/>
+<junction x="177.8" y="167.64"/>
 </segment>
 <segment>
@@
 <pinref part="GND15" gate="1" pin="GND"/>
 <wire x1="198.12" y1="73.66" x2="203.2" y2="73.66" width="0.1524" layer="91"/>
-<wire x1="203.2" y1="73.66" x2="203.2" y2="71.12" width="0.1524" layer="91"/>
+<wire x1="203.2" y1="73.66" x2="203.2" y2="66.04" width="0.1524" layer="91"/>
 <pinref part="JP3" gate="G$1" pin="2"/>
+<pinref part="R35" gate="G$1" pin="1"/>
+<wire x1="203.2" y1="66.04" x2="203.2" y2="63.5" width="0.1524" layer="91"/>
+<wire x1="228.6" y1="68.58" x2="228.6" y2="66.04" width="0.1524" layer="91"/>
+<wire x1="228.6" y1="66.04" x2="203.2" y2="66.04" width="0.1524" layer="91"/>
+<junction x="203.2" y="66.04"/>
 </segment>
 <segment>
@@
 <pinref part="U5" gate="G$1" pin="T+"/>
 <pinref part="TC-K" gate="G$1" pin="2"/>
-<wire x1="185.42" y1="182.88" x2="198.12" y2="182.88" width="0.1524" layer="91"/>
+<wire x1="167.64" y1="182.88" x2="180.34" y2="182.88" width="0.1524" layer="91"/>
 </segment>
 </net>
 <net name="N$11" class="0">
 <segment>
-<wire x1="185.42" y1="180.34" x2="187.96" y2="180.34" width="0.1524" layer="91"/>
-<wire x1="187.96" y1="180.34" x2="187.96" y2="177.8" width="0.1524" layer="91"/>
+<wire x1="167.64" y1="180.34" x2="170.18" y2="180.34" width="0.1524" layer="91"/>
+<wire x1="170.18" y1="180.34" x2="170.18" y2="177.8" width="0.1524" layer="91"/>
 <pinref part="U5" gate="G$1" pin="T-"/>
-<wire x1="187.96" y1="177.8" x2="198.12" y2="177.8" width="0.1524" layer="91"/>
+<wire x1="170.18" y1="177.8" x2="180.34" y2="177.8" width="0.1524" layer="91"/>
 <pinref part="TC-K" gate="G$1" pin="1"/>
 </segment>
@@
 <segment>
 <pinref part="U5" gate="G$1" pin="SO"/>
-<wire x1="218.44" y1="182.88" x2="220.98" y2="182.88" width="0.1524" layer="91"/>
-<label x="220.98" y="182.88" size="1.016" layer="95" xref="yes"/>
+<wire x1="200.66" y1="182.88" x2="203.2" y2="182.88" width="0.1524" layer="91"/>
+<label x="203.2" y="182.88" size="1.016" layer="95" xref="yes"/>
 </segment>
 <segment>
@@
 <segment>
 <pinref part="U5" gate="G$1" pin="SCK"/>
-<wire x1="218.44" y1="180.34" x2="220.98" y2="180.34" width="0.1524" layer="91"/>
-<label x="220.98" y="180.34" size="1.016" layer="95" xref="yes"/>
+<wire x1="200.66" y1="180.34" x2="203.2" y2="180.34" width="0.1524" layer="91"/>
+<label x="203.2" y="180.34" size="1.016" layer="95" xref="yes"/>
 </segment>
 <segment>
@@
 <segment>
 <pinref part="U5" gate="G$1" pin="/CS"/>
+<wire x1="200.66" y1="177.8" x2="218.44" y2="177.8" width="0.1524" layer="91"/>
+<label x="220.98" y="177.8" size="1.016" layer="95" xref="yes"/>
+<pinref part="R34" gate="G$1" pin="1"/>
 <wire x1="218.44" y1="177.8" x2="220.98" y2="177.8" width="0.1524" layer="91"/>
-<label x="220.98" y="177.8" size="1.016" layer="95" xref="yes"/>
+<wire x1="218.44" y1="180.34" x2="218.44" y2="177.8" width="0.1524" layer="91"/>
+<junction x="218.44" y="177.8"/>
 </segment>
 </net>
@@
 <segment>
 <pinref part="U5" gate="G$1" pin="VCC"/>
-<wire x1="198.12" y1="185.42" x2="195.58" y2="185.42" width="0.1524" layer="91"/>
-<wire x1="195.58" y1="185.42" x2="195.58" y2="187.96" width="0.1524" layer="91"/>
-<label x="195.58" y="187.96" size="1.016" layer="95" rot="R90" xref="yes"/>
+<wire x1="180.34" y1="185.42" x2="177.8" y2="185.42" width="0.1524" layer="91"/>
+<wire x1="177.8" y1="185.42" x2="177.8" y2="195.58" width="0.1524" layer="91"/>
+<label x="177.8" y="198.12" size="1.016" layer="95" rot="R90" xref="yes"/>
 <pinref part="C9" gate="G$1" pin="1"/>
-<wire x1="195.58" y1="185.42" x2="193.04" y2="185.42" width="0.1524" layer="91"/>
-<wire x1="193.04" y1="185.42" x2="193.04" y2="175.26" width="0.1524" layer="91"/>
-<junction x="195.58" y="185.42"/>
+<wire x1="177.8" y1="195.58" x2="177.8" y2="198.12" width="0.1524" layer="91"/>
+<wire x1="177.8" y1="185.42" x2="175.26" y2="185.42" width="0.1524" layer="91"/>
+<wire x1="175.26" y1="185.42" x2="175.26" y2="175.26" width="0.1524" layer="91"/>
+<junction x="177.8" y="185.42"/>
+<pinref part="R34" gate="G$1" pin="2"/>
+<wire x1="177.8" y1="195.58" x2="218.44" y2="195.58" width="0.1524" layer="91"/>
+<wire x1="218.44" y1="195.58" x2="218.44" y2="190.5" width="0.1524" layer="91"/>
+<junction x="177.8" y="195.58"/>
+<wire x1="177.8" y1="195.58" x2="218.44" y2="195.58" width="0.1524" layer="91"/>
 </segment>
 <segment>
@@
 <wire x1="246.38" y1="83.82" x2="243.84" y2="83.82" width="0.1524" layer="91"/>
 <wire x1="246.38" y1="83.82" x2="246.38" y2="81.28" width="0.1524" layer="91"/>
-<wire x1="246.38" y1="81.28" x2="198.12" y2="81.28" width="0.1524" layer="91"/>
+<wire x1="246.38" y1="81.28" x2="228.6" y2="81.28" width="0.1524" layer="91"/>
 <junction x="246.38" y="83.82"/>
 <pinref part="JP3" gate="G$1" pin="5"/>
-</segment>
-</net>
+<pinref part="R35" gate="G$1" pin="2"/>
+<wire x1="228.6" y1="81.28" x2="198.12" y2="81.28" width="0.1524" layer="91"/>
+<wire x1="228.6" y1="81.28" x2="228.6" y2="78.74" width="0.1524" layer="91"/>
+<junction x="228.6" y="81.28"/>
+</segment>
+</net>

Commit message: added disconnect for operation in string
Parts:
- added K1: AZ8-FORM-C, relay:AZ8-FORM-C
- added STRING: (no value), holla:M02-6.35MM
Connections:
- new net N$20: K1-1.P, STRING.2
- net GND: now also K1-1.S, STRING.1
- net VPANEL2: now also K1-1.O
Other:
- note added: "+"
- note added: "-"
- note added: "1.2mOhm"
- note added: "Current Sensor"
- note added: "Current Sensor Scaling"
- note added: "DISCONNECT"
- note added: "FET Gate Driver"
- note added: "FLOATING GND"
- note added: "LOAD"
- note added: "N-CH MOSFET Array"
- note added: "PANEL"
- note added: "Panel Voltage Scaling"
- note added: "TEST PANEL"
- note added: "need arc protection"
- moved on the sheet: C1, C2, C20, C3, C4, C5, C6, C7, C8, D1, D11, D2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

Commit message: added dual-coil latching relay and 23017 I/O port for future battery charger control
Parts:
- added IC1: MCP23017ML, microchip:MCP23017ML
- K1: value AZ8-FORM-C -> (none); device relay:AZ8-FORM-C -> holla:RELAY-LATCHING-DUAL-1FORMC-5MM-16A
Connections:
- removed net DISPLAYRESET: A1.P$31, DISP1.RESET, JP3.5, R35.2
- new net PERIPHERALRESET: A1.P$31, DISP1.RESET, IC1.!RESET, JP3.5, R35.2
- net GND: now also IC1.A0, IC1.A1, IC1.A2, IC1.VSS, K1-1.NO; no longer K1-1.S
- net I2C_SCL: now also IC1.SCL
- net I2C_SDA: now also IC1.SDA
- net N$20: now also K1-1.W; no longer K1-1.P
- net V3.3: now also IC1.VDD
- net VPANEL2: now also K1-1.NC; no longer K1-1.O
Other:
- note added: "Battery Charger Control AMUX Select"
- note added: "DUT"
- note added: "MOSFET Array Gate Driver"
- note added: "Panel Current Sensor Scaling"
- note added: "RESET=CONNECT"
- note added: "SET=DISCONNECT"
- note added: "put reverse voltage clamp here"
- note removed: "Current Sensor Scaling"
- note removed: "FET Gate Driver"
- moved on the sheet: C1, C2, C20, C3, C4, C5, C6, C7, C8, D1, D11, D2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

Commit message: fixed a bunch of top silk errors here and there
Parts:
- removed GOLD_ORB_SM1: LOGO-OSHW_GOLD_ORB_MED, holla:LOGO-OSHW_GOLD_ORB_MED
- added LOGO1: LOGO-OSHWL, holla:LOGO-OSHWL
Changed lines of the file:
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@@
 <part name="A1" library="TI-CC3200" deviceset="CC3200-LAUNCHXL-BOOSTERPACK" device="" value="CC3200-LAUNCHXL-BOOSTERPACK"/>
 <part name="PANEL" library="holla" deviceset="M02" device="-6.35MM"/>
-<part name="Q1" library="holla" deviceset="1984620" device="" value=""/>
-<part name="Q2" library="holla" deviceset="1984620" device="" value=""/>
-<part name="Q3" library="holla" deviceset="1984620" device="" value=""/>
-<part name="Q4" library="holla" deviceset="1984620" device="" value=""/>
-<part name="Q5" library="holla" deviceset="1984620" device="" value=""/>
-<part name="Q6" library="holla" deviceset="1984620" device="" value=""/>
-<part name="Q7" library="holla" deviceset="1984620" device="" value=""/>
-<part name="Q8" library="holla" deviceset="1984620" device="" value=""/>
+<part name="Q1" library="holla" deviceset="1984620" device="" value="1984620"/>
+<part name="Q2" library="holla" deviceset="1984620" device="" value="1984620"/>
+<part name="Q3" library="holla" deviceset="1984620" device="" value="1984620"/>
+<part name="Q4" library="holla" deviceset="1984620" device="" value="1984620"/>
+<part name="Q5" library="holla" deviceset="1984620" device="" value="1984620"/>
+<part name="Q6" library="holla" deviceset="1984620" device="" value="1984620"/>
+<part name="Q7" library="holla" deviceset="1984620" device="" value="1984620"/>
+<part name="Q8" library="holla" deviceset="1984620" device="" value="1984620"/>
 <part name="U1" library="holla" deviceset="ACS712" device="" value="20"/>
 <part name="GND1" library="holla" deviceset="GND" device=""/>
@@
 <part name="R7" library="holla" deviceset="R" device="-US_R0603" value="1K"/>
 <part name="C5" library="holla" deviceset="C" device="-USC0603" value=".1u"/>
-<part name="U3" library="holla" deviceset="DAC_MCP4725" device="SOT" value=""/>
+<part name="U3" library="holla" deviceset="DAC_MCP4725" device="SOT" value="DAC_MCP4725SOT"/>
 <part name="GND5" library="holla" deviceset="GND" device=""/>
 <part name="C6" library="holla" deviceset="C" device="-USC0603" value=".1u"/>
@@
 <part name="GND8" library="holla" deviceset="GND" device=""/>
 <part name="IPANEL" library="holla" deviceset="TESTPOINT" device="THRU" value=""/>
-<part name="PHOTOCELL" library="holla" deviceset="1984617" device="" value=""/>
+<part name="PHOTOCELL" library="holla" deviceset="1984617" device="" value="1984617"/>
 <part name="R13" library="holla" deviceset="R" device="-US_R0603" value="47K"/>
 <part name="GND9" library="holla" deviceset="GND" device=""/>
@@
 <part name="GND14" library="holla" deviceset="GND" device=""/>
 <part name="GND15" library="holla" deviceset="GND" device=""/>
-<part name="1WIRE" library="holla" deviceset="1984620" device="" value=""/>
+<part name="1WIRE" library="holla" deviceset="1984620" device="" value="1984620"/>
 <part name="GND17" library="holla" deviceset="GND" device=""/>
 <part name="R24" library="holla" deviceset="R" device="-US_R0603" value="1K"/>
@@
 <part name="JP1" library="holla" deviceset="FIDUCIAL" device="UFIDUCIAL"/>
 <part name="JP2" library="holla" deviceset="FIDUCIAL" device="UFIDUCIAL"/>
-<part name="F1" library="holla" deviceset="FUSE-HOLDER" device="-3557-2" value=""/>
+<part name="F1" library="holla" deviceset="FUSE-HOLDER" device="-3557-2" value="FUSE-HOLDER-3557-2"/>
 <part name="D2" library="holla" deviceset="ZENER" device="-SOD323" value="2.0"/>
 <part name="D3" library="holla" deviceset="ZENER" device="-SOD323" value="2.0"/>
@@
 <part name="SCL" library="holla" deviceset="TESTPOINT" device="THRU" value=""/>
 <part name="SDA" library="holla" deviceset="TESTPOINT" device="THRU" value=""/>
-<part name="GOLD_ORB_SM1" library="holla" deviceset="LOGO-OSHW" device="_GOLD_ORB_MED"/>
 <part name="C26" library="holla" deviceset="C" device="-USC0603" value=".1u"/>
 <part name="U12" library="holla" deviceset="IRDETECTOR" device="-TSOP6X"/>
@@
 <part name="IC1" library="microchip" deviceset="MCP23017" device="ML"/>
 <part name="GND29" library="holla" deviceset="GND" device=""/>
+<part name="LOGO1" library="holla" deviceset="LOGO-OSHW" device="L" value="LOGO-OSHWL"/>
 </parts>
 <sheets>
@@
 <instance part="JP1" gate="G$1" x="175.26" y="40.64"/>
 <instance part="JP2" gate="G$1" x="180.34" y="40.64"/>
-<instance part="GOLD_ORB_SM1" gate="G$1" x="256.54" y="48.26"/>
 <instance part="IC1" gate="G$1" x="71.12" y="78.74"/>
 <instance part="GND29" gate="1" x="55.88" y="53.34"/>
+<instance part="LOGO1" gate="G$1" x="256.54" y="48.26"/>
 </instances>
 <busses>

Commit message: initial add for src little tweaks to the board added lines to board design notes file
Parts:
- R1: value 33k -> 33K
- Y1: value 32.768KHz -> 32.768KHz-6pF
Connections:
- net 1WIRE renamed ONEWIRE
- net V3.3SCALED renamed V3P3SCALED
Changed lines of the file:
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@@
 <part name="GND2" library="holla" deviceset="GND" device=""/>
 <part name="C1" library="holla" deviceset="C" device="-USC0603" value=".1u"/>
-<part name="R1" library="holla" deviceset="R" device="-US_R0603" value="33k"/>
+<part name="R1" library="holla" deviceset="R" device="-US_R0603" value="33K"/>
 <part name="R2" library="holla" deviceset="R" device="-US_R0603" value="1K"/>
 <part name="C2" library="holla" deviceset="C" device="-USC0603" value="10n"/>
@@
 <part name="C24" library="holla" deviceset="C" device="-USC0603" value=".1u"/>
 <part name="GND26" library="holla" deviceset="GND" device=""/>
-<part name="Y1" library="holla" deviceset="CRYSTAL32-SMD" device="ABS25" value="32.768KHz"/>
+<part name="Y1" library="holla" deviceset="CRYSTAL32-SMD" device="ABS25" value="32.768KHz-6pF"/>
 <part name="C25" library="holla" deviceset="C" device="-SUPER-10MM" value="0.33F"/>
 <part name="BATT" library="holla" deviceset="M04" device="-B4B-XH-VERT"/>
@@
 </segment>
 </net>
-<net name="1WIRE" class="0">
+<net name="ONEWIRE" class="0">
 <segment>
 <pinref part="A1" gate="G$1" pin="P$11"/>
@@
 </segment>
 </net>
-<net name="1WIRE" class="0">
+<net name="ONEWIRE" class="0">
 <segment>
 <pinref part="1WIRE" gate="G$1" pin="2"/>
@@
 </segment>
 </net>
-<net name="V3.3SCALED" class="0">
+<net name="V3P3SCALED" class="0">
 <segment>
 <pinref part="U7" gate="G$1" pin="Y4"/>
