File: board/solohm.brd (EAGLE design)
At the start: 99 x 99 mm, 113 parts, among them IC1 MCP23017ML, Q1 1984620, Q2 1984620, Q3 1984620, Q4 1984620, Q5 1984620, Q6 1984620, Q7 1984620, Q8 1984620, U1 20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

Commit message: fixed amux ground islands ino has functional vbatt sensing
Routing:
- net GND: vias 27 -> 28
Changed lines of the file:
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@@
 <contactref element="IC1" pad="13"/>
 <contactref element="IC1" pad="6"/>
+<via x="24.511" y="18.542" extent="1-16" drill="0.6" shape="square"/>
 <wire x1="-26.401" y1="-31.402" x2="-27.051" y2="-31.402" width="0" layer="19" extent="1-1"/>
 <wire x1="-25.751" y1="-31.402" x2="-26.401" y2="-31.402" width="0" layer="19" extent="1-1"/>
@@
 <wire x1="5.167" y1="-31.055" x2="5.167" y2="-23.555" width="0" layer="19" extent="1-1"/>
 <wire x1="5.08" y1="13.97" x2="-18.923" y2="-8.636" width="0" layer="19" extent="1-1"/>
-<wire x1="22.225" y1="19.625" x2="25.908" y2="22.186" width="0" layer="19" extent="1-1"/>
-<wire x1="15.875" y1="14.04" x2="21.209" y2="14.39" width="0" layer="19" extent="1-1"/>
 <wire x1="73.66" y1="9.105" x2="62.865" y2="7.62" width="0" layer="19" extent="1-1"/>
 </signal>
@@
 <wire x1="25.82" y1="20.574" x2="25.908" y2="20.486" width="0.3048" layer="1"/>
 <wire x1="10.668" y1="12.358" x2="10.668" y2="11.43" width="0.3048" layer="1"/>
-<wire x1="10.668" y1="11.43" x2="11.176" y2="10.922" width="0.3048" layer="1"/>
-<wire x1="11.176" y1="10.922" x2="21.59" y2="10.922" width="0.3048" layer="1"/>
-<wire x1="21.59" y1="10.922" x2="25.908" y2="10.922" width="0.3048" layer="1"/>
-<wire x1="25.908" y1="10.922" x2="26.162" y2="11.176" width="0.3048" layer="1"/>
-<wire x1="26.162" y1="11.176" x2="26.162" y2="20.232" width="0.3048" layer="1"/>
+<wire x1="10.668" y1="11.43" x2="11.938" y2="9.906" width="0.3048" layer="1"/>
+<wire x1="11.938" y1="9.906" x2="21.082" y2="9.906" width="0.3048" layer="1"/>
+<wire x1="21.082" y1="9.906" x2="21.844" y2="9.906" width="0.3048" layer="1"/>
+<wire x1="21.844" y1="9.906" x2="24.892" y2="9.906" width="0.3048" layer="1"/>
+<wire x1="24.892" y1="9.906" x2="26.162" y2="11.811" width="0.3048" layer="1"/>
+<wire x1="26.162" y1="11.811" x2="26.162" y2="20.232" width="0.3048" layer="1"/>
 <wire x1="26.162" y1="20.232" x2="25.908" y2="20.486" width="0.3048" layer="1"/>
-<wire x1="21.661" y1="7.62" x2="21.661" y2="10.851" width="0.3048" layer="1"/>
-<wire x1="21.661" y1="10.851" x2="21.59" y2="10.922" width="0.3048" layer="1"/>
+<wire x1="21.661" y1="7.62" x2="21.661" y2="9.723" width="0.2032" layer="1"/>
+<wire x1="21.661" y1="9.723" x2="21.844" y2="9.906" width="0.2032" layer="1"/>
 </signal>
 <signal name="VBATT2SCALED">
